File: schematic/Kicad/Basic_setup/Basic_Setup.kicad_sch (KiCad schematic)
At the start: 38 parts, among them J1 AUDIO, Y1 32.768kHz

Commit message: Doc
Parts:
- removed AE1: Antenna, symbol Device:Antenna
- removed C1, C12, C3, C4, C5, C8: 0.1uF, symbol Device:C
- removed C10: 33pF, symbol Device:C
- removed C11: 18pF, symbol Device:C
- removed C2: 1uF, symbol Device:C
- removed C6, C7: 22pF, symbol Device:C
- removed C9: 10pF, symbol Device:C
- removed D1: LED, symbol Device:LED
- removed J1: AUDIO, symbol Connector:Conn_01x01_Pin
- removed L1: L_Ferrite, symbol Device:L_Ferrite
- removed L2: 100nH, symbol Device:L
- removed R14: 2.2K, symbol Device:R
- removed R15: 220R, symbol Device:R
- removed R16: 1K, symbol Device:R
- removed R17: 10K, symbol Device:R
- removed TUNE: 100K, SI4844_01:POT-PTH-ALPS, symbol SI4844:POTENTIOMETER-PTH-9MM-1/20W-20%
- removed U1: ~, BKXXXX:BK1198, symbol SI48XX:BK1198
- removed Y1: 32.768kHz, symbol Device:Crystal
- R1: value 10K -> 67K
- R2: value 60K -> 190K
- R3: value 60K -> 40K
- R4: value 20K -> 10K
- R5: value 20K -> 30K
Other:
- note added: "257K"
- note added: "297K"
- note added: "307K"
- note added: "337K"
- note added: "357K"
- note added: "AM4"
- note added: "FM/FM3"
- note added: "Si4825 BAND(PIN 4)"
- note removed: "FM"
- note removed: "MW"
- note removed: "R1 - FM: 87 - 108MHz R1 - MW: 520 - 1710kHz R3 - SW1: 4.70 - 5.10MHz R4 - SW2: 5.50 - 6.50MHz R5 - SW3: 6.70 - 7.70MHz R6 - SW4: 9.10 - 10.10MHz R7 - SW5: 11.40 - 12.40MHz R8 - SW6: 13.40 - 14.30MHz R9 - SW7: 15.00 - 16.00MHz R10- SW8: 17.00 - 18.00MHz R11- SW9: 16.98 - 18.10MHz R12- SW10: 21.10 - 22.10MHz"
- note removed: "RST"
- note removed: "SW1"
- note removed: "SW2"
- moved on the sheet: BAND_SELECT, R1, R10, R11, R12, R13, R2, R3, R4, R5, R6, R7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
