File: schematic/Kicad/si4825_basic_setup/si4825_basic_setup.kicad_sch (KiCad schematic)
At the start: 30 parts, among them J1 AudioJack2, Y1 32.768kHz

Commit message: Doc
Parts:
- added R15: 10K, symbol Device:R
- added SW1: W_N, symbol Switch:SW_SPDT
Connections:
- net +3.3V: now also R15.2
- net at U1.1 (LNA_EN): now also SW1.2 (B)
- new net: R15.1, SW1.1 (A)
Other:
- note added: "Narrow Band"
- note added: "Optional"
- note added: "The LNA_EN pin allows the selection of Wide or Narrow band. Refer to the SI4825 documentation for more details."
- note added: "Wide Band"
Changed lines of the file:
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@@
+    (stroke (width 0) (type default))
+  )
+  (wire (pts (xy 120.65 93.98) (xy 120.65 100.33))
     (stroke (width 0) (type default))
   )
@@
     (stroke (width 0) (type default))
   )
-  (wire (pts (xy 125.73 80.01) (xy 125.73 82.55))
+  (wire (pts (xy 125.73 80.01) (xy 125.73 81.28))
     (stroke (width 0) (type default))
   )
@@
     (stroke (width 0) (type default))
   )
+  (wire (pts (xy 118.11 93.98) (xy 120.65 93.98))
+    (stroke (width 0) (type default))
+  )
+  (wire (pts (xy 120.65 107.95) (xy 120.65 109.22))
+    (stroke (width 0) (type default))
+  )
   (wire (pts (xy 87.63 48.26) (xy 87.63 40.64))
     (stroke (width 0) (type default))
@@
     (stroke (width 0) (type default))
   )
+  (wire (pts (xy 102.87 91.44) (xy 107.95 91.44))
+    (stroke (width 0) (type default))
+  )
   (wire (pts (xy 62.23 22.86) (xy 62.23 45.72))
     (stroke (width 0) (type default))
@@
   (wire (pts (xy 91.44 151.13) (xy 91.44 152.4))
     (stroke (width 0) (type default))
+  )
+  (rectangle (start 106.68 85.09) (end 133.35 114.3)
+    (stroke (width 0) (type default))
+    (fill (type none))
   )
   (text "SW7" (at 83.82 38.1 90)
@@
     (effects (font (size 1.27 1.27)) (justify left bottom))
   )
+  (text "Wide Band" (at 121.92 96.52 0)
+    (effects (font (size 1.27 1.27)) (justify left bottom))
+  )
   (text "437K" (at 129.54 30.48 90)
     (effects (font (size 1.27 1.27)) (justify left bottom))
@@
   )
   (text "307K" (at 76.2 30.48 90)
+    (effects (font (size 1.27 1.27)) (justify left bottom))
+  )
+  (text "The LNA_EN pin allows the selection of Wide or Narrow band. \nRefer to the SI4825 documentation for more details."
+    (at 135.89 143.51 0)
     (effects (font (size 1.27 1.27)) (justify left bottom))
   )
@@
     (effects (font (face "Courier New") (size 1.27 1.27) (thickness 0.254) bold) (justify left bottom))
   )
+  (text "Narrow Band" (at 119.38 90.17 0)
+    (effects (font (size 1.27 1.27)) (justify left bottom))
+  )
+  (text "Optional" (at 106.68 85.09 0)
+    (effects (font (size 1.27 1.27)) (justify left bottom))
+  )
   (text "387K" (at 106.68 30.48 90)
     (effects (font (size 1.27 1.27)) (justify left bottom))
@@
     )
   )
-  (symbol (lib_id "power:GND") (at 125.73 82.55 0) (unit 1)
-    (in_bom yes) (on_board yes) (dnp no) (fields_autoplaced)
-    (property "Reference" "#PWR02" (at 125.73 88.9 0)
-      (effects (font (size 1.27 1.27)) hide)
-    )
-    (property "Value" "GND" (at 125.73 87.63 0)
-      (effects (font (size 1.27 1.27)))
-    )
-    (property "Footprint" "" (at 125.73 82.55 0)
-      (effects (font (size 1.27 1.27)) hide)
-    )
-    (property "Datasheet" "" (at 125.73 82.55 0)
+  (symbol (lib_id "power:GND") (at 125.73 81.28 0) (unit 1)
+    (in_bom yes) (on_board yes) (dnp no)
+    (property "Reference" "#PWR02" (at 125.73 87.63 0)
+      (effects (font (size 1.27 1.27)) hide)
+    )
+    (property "Value" "GND" (at 128.27 78.74 0)
+      (effects (font (size 1.27 1.27)))
+    )
+    (property "Footprint" "" (at 125.73 81.28 0)
+      (effects (font (size 1.27 1.27)) hide)
+    )
+    (property "Datasheet" "" (at 125.73 81.28 0)
       (effects (font (size 1.27 1.27)) hide)
     )
@@
     )
   )
+  (symbol (lib_id "power:+3.3V") (at 120.65 109.22 180) (unit 1)
+    (in_bom yes) (on_board yes) (dnp no)
+    (property "Reference" "#PWR014" (at 120.65 105.41 0)
+      (effects (font (size 1.27 1.27)) hide)
+    )
+    (property "Value" "+3.3V" (at 123.19 113.03 0)
+      (effects (font (size 1.27 1.27)))
+    )
+    (property "Footprint" "" (at 120.65 109.22 0)
+      (effects (font (size 1.27 1.27)) hide)
+    )
+    (property "Datasheet" "" (at 120.65 109.22 0)
+      (effects (font (size 1.27 1.27)) hide)
+    )
+    (pin "1")
+    (instances
+      (project "si4825_basic_setup"
+        (path "/cf4feedd-3416-459a-83d0-42e924d6c0b9"
+          (reference "#PWR014") (unit 1)
+        )
+      )
+    )
+  )
   (symbol (lib_id "Device:R") (at 66.04 22.86 270) (unit 1)
     (in_bom yes) (on_board yes) (dnp no) (fields_autoplaced)
@@
         (path "/cf4feedd-3416-459a-83d0-42e924d6c0b9"
           (reference "R3") (unit 1)
+        )
+      )
+    )
+  )
+  (symbol (lib_id "Device:R") (at 120.65 104.14 0) (unit 1)
+    (in_bom yes) (on_board yes) (dnp no) (fields_autoplaced)
+    (property "Reference" "R15" (at 123.19 102.87 0)
+      (effects (font (size 1.27 1.27)) (justify left))
+    )
+    (property "Value" "10K" (at 123.19 105.41 0)
+      (effects (font (size 1.27 1.27)) (justify left))
+    )
+    (property "Footprint" "" (at 118.872 104.14 90)
+      (effects (font (size 1.27 1.27)) hide)
+    )
+    (property "Datasheet" "~" (at 120.65 104.14 0)
+      (effects (font (size 1.27 1.27)) hide)
+    )
+    (pin "1")
+    (pin "2")
+    (instances
+      (project "si4825_basic_setup"
+        (path "/cf4feedd-3416-459a-83d0-42e924d6c0b9"
+          (reference "R15") (unit 1)
         )
       )
@@
   )
   (symbol (lib_id "SI4844:POTENTIOMETER-PTH-9MM-1/20W-20%") (at 118.11 80.01 90) (unit 1)
-    (in_bom yes) (on_board yes) (dnp no) (fields_autoplaced)
-    (property "Reference" "VR1" (at 118.11 83.82 90)
+    (in_bom yes) (on_board yes) (dnp no)
+    (property "Reference" "VR1" (at 118.11 82.55 90)
       (effects (font (size 1.778 1.778)))
     )
@@
   )
   (symbol (lib_id "Device:C") (at 119.38 119.38 270) (unit 1)
-    (in_bom yes) (on_board yes) (dnp no) (fields_autoplaced)
-    (property "Reference" "C1" (at 119.38 111.76 90)
-      (effects (font (size 1.27 1.27)))
-    )
-    (property "Value" "1UF" (at 119.38 114.3 90)
+    (in_bom yes) (on_board yes) (dnp no)
+    (property "Reference" "C1" (at 116.84 124.46 90)
+      (effects (font (size 1.27 1.27)))
+    )
+    (property "Value" "1UF" (at 120.65 124.46 90)
       (effects (font (size 1.27 1.27)))
     )
@@
         (path "/cf4feedd-3416-459a-83d0-42e924d6c0b9"
           (reference "C1") (unit 1)
+        )
+      )
+    )
+  )
+  (symbol (lib_id "Switch:SW_SPDT") (at 113.03 91.44 0) (mirror x) (unit 1)
+    (in_bom yes) (on_board yes) (dnp no)
+    (property "Reference" "SW1" (at 113.03 99.06 0)
+      (effects (font (size 1.27 1.27)))
+    )
+    (property "Value" "W_N" (at 113.03 96.52 0)
+      (effects (font (size 1.27 1.27)))
+    )
+    (property "Footprint" "" (at 113.03 91.44 0)
+      (effects (font (size 1.27 1.27)) hide)
+    )
+    (property "Datasheet" "~" (at 113.03 91.44 0)
+      (effects (font (size 1.27 1.27)) hide)
+    )
+    (pin "1")
+    (pin "2")
+    (pin "3")
+    (instances
+      (project "si4825_basic_setup"
+        (path "/cf4feedd-3416-459a-83d0-42e924d6c0b9"
+          (reference "SW1") (unit 1)
         )
       )
@@
   )
   (symbol (lib_id "SI48XX:SI4825") (at 104.14 105.41 270) (unit 1)
-    (in_bom yes) (on_board yes) (dnp no) (fields_autoplaced)
-    (property "Reference" "U1" (at 107.95 102.87 90)
+    (in_bom yes) (on_board yes) (dnp no)
+    (property "Reference" "U1" (at 101.6 106.68 90)
       (effects (font (size 1.27 1.27)) (justify left))
     )
