File: schematic/Kicad/si4825_Narrow_Wide_Band_setup/si4825_Narrow_Wide_Band_setup.kicad_sch (KiCad schematic)
At the start: 12 parts, among them SW1 W_N, SW2 BAND_SWITCH

Commit message: Doc
Connections:
- net GND: no longer U1.15 (GND)
Changed lines of the file:
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@@
-    (stroke (width 0) (type default))
-  )
-  (wire (pts (xy 78.74 97.79) (xy 78.74 101.6))
     (stroke (width 0) (type default))
   )
@@
     (stroke (width 0) (type default))
   )
-  (wire (pts (xy 66.04 66.04) (xy 66.04 69.85))
-    (stroke (width 0) (type default))
-  )
   (wire (pts (xy 93.98 25.4) (xy 93.98 50.8))
     (stroke (width 0) (type default))
@@
   )
   (wire (pts (xy 59.69 31.75) (xy 71.12 31.75))
-    (stroke (width 0) (type default))
-  )
-  (wire (pts (xy 68.58 50.8) (xy 68.58 69.85))
     (stroke (width 0) (type default))
   )
@@
         )
       )
-    )
-  )
-  (symbol (lib_id "power:GND") (at 78.74 101.6 0) (unit 1)
-    (in_bom yes) (on_board yes) (dnp no) (fields_autoplaced)
-    (property "Reference" "#PWR04" (at 78.74 107.95 0)
-      (effects (font (size 1.27 1.27)) hide)
-    )
-    (property "Value" "GND" (at 78.74 106.68 0)
-      (effects (font (size 1.27 1.27)) hide)
-    )
-    (property "Footprint" "" (at 78.74 101.6 0)
-      (effects (font (size 1.27 1.27)) hide)
-    )
-    (property "Datasheet" "" (at 78.74 101.6 0)
-      (effects (font (size 1.27 1.27)) hide)
-    )
-    (pin "1")
-    (instances
-      (project "si4825_Narrow_Wide_Band_setup"
-        (path "/cf4feedd-3416-459a-83d0-42e924d6c0b9"
-          (reference "#PWR04") (unit 1)
-        )
-      )
