File: schematic/Kicad/si4825_band_setup_example/si4825_band_setup_example.kicad_sch (KiCad schematic)
At the start: 14 parts

Commit message: Doc
Parts:
- R10, R12, R7: value 20K -> 10K
- R13: value 10K -> 53K
Other:
- note added: "367K"
- note added: "387K"
- note added: "407K"
- note added: "417K"
- note added: "437K"
- note added: "447K"
- note added: "SW12"
- note added: "SW14"
- note added: "SW15"
- note added: "SW17"
- note added: "SW18"
- note added: "Si4825 TUNE1(PIN 2)"
- note added: "| Band Name | Band Frequency Range | | ---------- | -------------------------- | | FM3 | 87-108 MHz (75 µs) | | AM4 | 522-1728 kHz/520-1730 kHz | | SW3-Narrow | 3.90-4.00 MHz | | SW4-Narrow | 4.75-5.06 MHz | | SW9-Narrow | 9.2-10 MHz | | SW10-Narrow| 11.45-12.25 MHz | | SW12-Narrow| 13.4-14.2 MHz | | SW14-Narrow| 15 -15.9 MHz | | SW15-Narrow| 17.1 -18 MHz | | SW17-Narrow| 21.2-22 MHz | | SW18-Nar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"
- note removed: "SW5"
- note removed: "SW6"
- note removed: "SW8"
- title: BK1198 BASIC SETUP - VOLTAGE DIVIDER VERSION (SW BAND) -> SI4825 Band setup example
- moved on the sheet: BAND_SELECT, R1, R10, R11, R12, R13, R2, R3, R4, R5, R6, R7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

Commit message: Doc
Parts:
- R12: value 10K -> 20K
- R2: value 190K -> 200K
- R3: value 40K -> 10K
- R4: value 10K -> 30K
- R6, R9: value 20K -> 10K
Other:
- note added: "267"
- note added: "277K"
- note added: "347K"
- note added: "397K"
- note added: "427K"
- note added: "AM5"
- note added: "SW1"
- note added: "SW13"
- note added: "SW16"
- note added: "SW8"
- note added: "| Band Name | Narrow Frequency Range | Wide Frequency Range | | ---------- | ------------------------| ---------------------- | | FM3 | 87-108 MHz (75 µs) | | | AM5 | 510-1750 kHz (10kHz) | | | SW1 | 2.30-2.49 MHz | 2.3-10.0 MHz | | SW4 | 4.75-5.06 MHz | 3.7-12.5 MHz | | SW8 | 7.1-7.6 MHz | 5.9-9.50 MHz | | SW9 | 9.2-10 MHz | 5.9-18.0 MHz | | SW10 | 11.45-12.25 MHz | 7.0-16.0 MHz | | SW12 | 13.4-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"
- note removed: "257K"
- note removed: "297K"
- note removed: "337K"
- note removed: "417K"
- note removed: "437K"
- note removed: "AM4"
- note removed: "SW15"
- note removed: "SW17"
- note removed: "SW3"
- note removed: "SW7"
- note removed: "| Band Name | Band Frequency Range | | ---------- | -------------------------- | | FM3 | 87-108 MHz (75 µs) | | AM4 | 522-1728 kHz/520-1730 kHz | | SW3-Narrow | 3.90-4.00 MHz | | SW4-Narrow | 4.75-5.06 MHz | | SW9-Narrow | 9.2-10 MHz | | SW10-Narrow| 11.45-12.25 MHz | | SW12-Narrow| 13.4-14.2 MHz | | SW14-Narrow| 15 -15.9 MHz | | SW15-Narrow| 17.1 -18 MHz | | SW17-Narrow| 21.2-22 MHz | | SW18-Nar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"
Changed lines of the file:
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@@
     (stroke (width 0) (type default))
   )
-  (text "SW7" (at 82.55 52.07 90)
+  (text "SW8" (at 82.55 52.07 90)
     (effects (font (size 1.27 1.27) (thickness 0.254) bold) (justify left bottom))
   )
@@
     (effects (font (size 1.27 1.27)) (justify left bottom))
   )
-  (text "437K" (at 128.27 44.45 90)
+  (text "427K" (at 128.27 44.45 90)
     (effects (font (size 1.27 1.27)) (justify left bottom))
   )
@@
     (effects (font (size 1.5 1.5) (thickness 0.3) bold) (justify left bottom))
   )
-  (text "337K" (at 82.55 44.45 90)
-    (effects (font (size 1.27 1.27)) (justify left bottom))
-  )
-  (text "SW15" (at 120.65 50.8 90)
+  (text "347K" (at 82.55 44.45 90)
+    (effects (font (size 1.27 1.27)) (justify left bottom))
+  )
+  (text "SW14" (at 120.65 50.8 90)
     (effects (font (size 1.27 1.27) (thickness 0.254) bold) (justify left bottom))
   )
@@
     (effects (font (size 1.27 1.27) (thickness 0.254) bold) (justify left bottom))
   )
-  (text "417K" (at 120.65 44.45 90)
+  (text "407K" (at 120.65 44.45 90)
     (effects (font (size 1.27 1.27)) (justify left bottom))
   )
@@
     (effects (font (size 1.27 1.27) (thickness 0.254) bold) (justify left bottom))
   )
-  (text "AM4" (at 59.69 52.07 90)
-    (effects (font (size 1.27 1.27) (thickness 0.254) bold) (justify left bottom))
-  )
-  (text "297K" (at 67.31 44.45 90)
+  (text "AM5" (at 59.69 52.07 90)
+    (effects (font (size 1.27 1.27) (thickness 0.254) bold) (justify left bottom))
+  )
+  (text "277K" (at 67.31 44.45 90)
     (effects (font (size 1.27 1.27)) (justify left bottom))
   )
@@
     (effects (font (size 1.27 1.27)) (justify left bottom))
   )
-  (text "407K" (at 113.03 44.45 90)
+  (text "397K" (at 113.03 44.45 90)
     (effects (font (size 1.27 1.27)) (justify left bottom))
   )
@@
     (effects (font (size 1.27 1.27)) (justify left bottom))
   )
-  (text "| Band Name  | Band Frequency Range       |\n| ---------- | -------------------------- |\n| FM3        | 87-108 MHz (75 µs)         | \n| AM4        | 522-1728 kHz/520-1730 kHz  |\n| SW3-Narrow | 3.90-4.00 MHz              |\n| SW4-Narrow | 4.75-5.06 MHz              |\n| SW9-Narrow | 9.2-10 MHz                 |\n| SW10-Narrow| 11.45-12.25 MHz            | \n| SW12-Narrow| 13.4-14.2 MHz              |\n| SW14-Narrow| 15 -15.9 MHz               |\n| SW15-Narrow| 17.1 -18 MHz               |\n| SW17-Narrow| 21.2-22 MHz                |\n| SW18-Narrow| 21.45-21.85 MHz            |\n\nSee Si4825 DEMO BOARD USER'S GUIDE for more details"
-    (at 16.51 101.6 0)
+  (text "| Band Name  | Narrow Frequency Range  | Wide Frequency Range   |\n| ---------- | ------------------------| ---------------------- |\n| FM3        | 87-108 MHz (75 µs)      |                        |\n| AM5        | 510-1750 kHz (10kHz)    |                        |\n| SW1        | 2.30-2.49 MHz           | 2.3-10.0 MHz           |\n| SW4        | 4.75-5.06 MHz           | 3.7-12.5 MHz           |\n| SW8        | 7.1-7.6 MHz             | 5.9-9.50 MHz           |\n| SW9        | 9.2-10 MHz              | 5.9-18.0 MHz           |\n| SW10       | 11.45-12.25 MHz         | 7.0-16.0 MHz           |\n| SW12       | 13.4-14.2 MHz           | 9.0-16.0 MHz           |\n| SW13       | 13.57-13.87 MHz         | 9.0-22.0 MHz           |\n| SW14       | 15 -15.9 MHz            | 9.5-18.0 MHz           |\n| SW16       | 17.48-17.9 MHz          | 10.0-22.0 MHz          |\n| SW18       | 21.45-21.85 MHz         | 18.0-28.5 MHz          |\n\nSee Si4825 DEMO BOARD USER'S GUIDE for more details"
+    (at 15.24 120.65 0)
     (effects (font (face "Courier New") (size 1.27 1.27) (thickness 0.254) bold) (justify left bottom))
   )
@@
     (effects (font (size 1.27 1.27)) (justify left bottom))
   )
-  (text "SW17" (at 128.27 50.8 90)
-    (effects (font (size 1.27 1.27) (thickness 0.254) bold) (justify left bottom))
-  )
-  (text "257K" (at 59.69 44.45 90)
-    (effects (font (size 1.27 1.27)) (justify left bottom))
-  )
-  (text "SW14" (at 113.03 50.8 90)
+  (text "SW16" (at 128.27 50.8 90)
+    (effects (font (size 1.27 1.27) (thickness 0.254) bold) (justify left bottom))
+  )
+  (text "267" (at 59.69 44.45 90)
+    (effects (font (size 1.27 1.27)) (justify left bottom))
+  )
+  (text "SW13" (at 113.03 50.8 90)
     (effects (font (size 1.27 1.27) (thickness 0.254) bold) (justify left bottom))
   )
@@
     (effects (font (size 1.27 1.27) (thickness 0.254) bold) (justify left bottom))
   )
-  (text "SW3" (at 67.31 52.07 90)
+  (text "SW1" (at 67.31 52.07 90)
     (effects (font (size 1.27 1.27) (thickness 0.254) bold) (justify left bottom))
   )
@@
       (effects (font (size 1.27 1.27)))
     )
-    (property "Value" "10K" (at 72.39 33.02 90)
+    (property "Value" "30K" (at 72.39 33.02 90)
       (effects (font (size 1.27 1.27)))
     )
@@
     (pin "2")
     (instances
-      (project "Basic_Setup"
+      (project "si4825_band_setup_example"
         (path "/cf4feedd-3416-459a-83d0-42e924d6c0b9"
           (reference "R4") (unit 1)
@@
     (pin "2")
     (instances
-      (project "Basic_Setup"
+      (project "si4825_band_setup_example"
         (path "/cf4feedd-3416-459a-83d0-42e924d6c0b9"
           (reference "R8") (unit 1)
@@
     (pin "2")
     (instances
-      (project "Basic_Setup"
+      (project "si4825_band_setup_example"
         (path "/cf4feedd-3416-459a-83d0-42e924d6c0b9"
           (reference "R10") (unit 1)
@@
       (effects (font (size 1.27 1.27)))
     )
-    (property "Value" "20K" (at 110.49 33.02 90)
+    (property "Value" "10K" (at 110.49 33.02 90)
       (effects (font (size 1.27 1.27)))
     )
@@
     (pin "2")
     (instances
-      (project "Basic_Setup"
+      (project "si4825_band_setup_example"
         (path "/cf4feedd-3416-459a-83d0-42e924d6c0b9"
           (reference "R9") (unit 1)
@@
       (effects (font (size 1.27 1.27)))
     )
-    (property "Value" "40K" (at 64.77 33.02 90)
+    (property "Value" "10K" (at 64.77 33.02 90)
       (effects (font (size 1.27 1.27)))
     )
@@
     (pin "2")
     (instances
-      (project "Basic_Setup"
+      (project "si4825_band_setup_example"
         (path "/cf4feedd-3416-459a-83d0-42e924d6c0b9"
           (reference "R3") (unit 1)
@@
       (effects (font (size 1.27 1.27)))
     )
-    (property "Value" "20K" (at 87.63 33.02 90)
+    (property "Value" "10K" (at 87.63 33.02 90)
       (effects (font (size 1.27 1.27)))
     )
@@
     (pin "2")
     (instances
-      (project "Basic_Setup"
+      (project "si4825_band_setup_example"
         (path "/cf4feedd-3416-459a-83d0-42e924d6c0b9"
           (reference "R6") (unit 1)
@@
     (pin "2")
     (instances
-      (project "Basic_Setup"
+      (project "si4825_band_setup_example"
         (path "/cf4feedd-3416-459a-83d0-42e924d6c0b9"
           (reference "R1") (unit 1)
@@
     (pin "9")
     (instances
-      (project "Basic_Setup"
+      (project "si4825_band_setup_example"
         (path "/cf4feedd-3416-459a-83d0-42e924d6c0b9"
           (reference "BAND_SELECT") (unit 1)
@@
     (pin "2")
     (instances
-      (project "Basic_Setup"
+      (project "si4825_band_setup_example"
         (path "/cf4feedd-3416-459a-83d0-42e924d6c0b9"
           (reference "R11") (unit 1)
@@
       (effects (font (size 1.27 1.27)))
     )
-    (property "Value" "190K" (at 57.15 33.02 90)
+    (property "Value" "200K" (at 57.15 33.02 90)
       (effects (font (size 1.27 1.27)))
     )
@@
     (pin "2")
     (instances
-      (project "Basic_Setup"
+      (project "si4825_band_setup_example"
         (path "/cf4feedd-3416-459a-83d0-42e924d6c0b9"
           (reference "R2") (unit 1)
@@
     (pin "2")
     (instances
-      (project "Basic_Setup"
+      (project "si4825_band_setup_example"
         (path "/cf4feedd-3416-459a-83d0-42e924d6c0b9"
           (reference "R5") (unit 1)
@@
       (effects (font (size 1.27 1.27)))
     )
-    (property "Value" "10K" (at 133.35 33.02 90)
+    (property "Value" "20K" (at 133.35 33.02 90)
       (effects (font (size 1.27 1.27)))
     )
@@
     (pin "2")
     (instances
-      (project "Basic_Setup"
+      (project "si4825_band_setup_example"
         (path "/cf4feedd-3416-459a-83d0-42e924d6c0b9"
           (reference "R12") (unit 1)
@@
     (pin "2")
     (instances
-      (project "Basic_Setup"
+      (project "si4825_band_setup_example"
         (path "/cf4feedd-3416-459a-83d0-42e924d6c0b9"
           (reference "R7") (unit 1)
@@
     (pin "2")
     (instances
-      (project "Basic_Setup"
+      (project "si4825_band_setup_example"
         (path "/cf4feedd-3416-459a-83d0-42e924d6c0b9"
           (reference "R13") (unit 1)
@@
     (pin "1")
     (instances
-      (project "Basic_Setup"
+      (project "si4825_band_setup_example"
         (path "/cf4feedd-3416-459a-83d0-42e924d6c0b9"
           (reference "#PWR01") (unit 1)
